Commit message: add board.obj to model and update urdf

File: project/panda_arm.urdf (robot description, URDF)
Before this commit: robot panda, 8 links, 7 joints
Links:
- link link7: geometry visual mesh filename=../../../model/panda/meshes/visual/Board.obj scale=0.4, 0.4, 0.4; visual mesh filename=../../../model/panda/meshes/visual/link7.obj

Commit message: added basketball court

File: project/panda_arm.urdf (robot description, URDF)
Before this commit: robot panda, 8 links, 7 joints
Links:
- link link7: geometry visual mesh filename=../../../model/mmp_panda/meshes/visual/Board.obj scale=0.4, 0.4, 0.4; visual mesh filename=../../../model/panda/meshes/visual/link7.obj
