Commit message: testing collision

File: project/kuka_iiwa1.urdf (robot description, URDF)
Before this commit: robot kuka_iiwa, 10 links, 9 joints
Links:
- removed link link8
- link link6: geometry visual mesh filename=../../../model/iiwa7/meshes/hand.obj scale=0.32 0.32 0.32; visual mesh filename=../../../model/iiwa7/meshes/link6.obj scale=1 1 1
- link link7: mass 1 -> 10; geometry visual box size=1 1 0.15
Joints:
- removed joint j7
- removed joint j8
