Commit message: modified wolrd and simviz

File: project/kuka_iiwa.urdf (robot description, URDF)
Before this commit: robot kuka_iiwa, 8 links, 7 joints
Links:
- link link6: geometry collision mesh filename=../../../model/iiwa7/meshes/launcher.obj scale=10 10 10; collision mesh filename=../../../model/iiwa7/meshes/link6.obj scale=1 1 1
Joints:
- joint j5: origin xyz=0.000000 0.000000 0.217003 rpy=0.000000 1.5000 0.000000 -> xyz=0.000000 0.000000 0.217003 rpy=0.000000 0.00 0.000000

File: project/mmp_panda.urdf (robot description, URDF)
Before this commit: robot mmp_panda, 11 links, 10 joints
Links:
- link base_link: geometry collision box size=0.4 0.4 0.2; visual mesh filename=../../../model/mmp_panda/meshes/visual/panda_BaseCombo.obj

Commit message: ?

File: project/kuka_iiwa.urdf (robot description, URDF)
Before this commit: robot kuka_iiwa, 8 links, 7 joints
Links:
- link link6: geometry collision mesh filename=../../../model/iiwa7/meshes/link6.obj scale=1 1 1; visual mesh filename=../../../model/iiwa7/meshes/hand.obj scale=0.32 0.32 0.32
Joints:
- joint j1: origin xyz=0.000000 0.000000 0.182500 rpy=0.000000 -0.500000 0.000000 -> xyz=0.000000 0.000000 0.182500 rpy=0.000000 -0.800000 0.000000
- joint j3: origin xyz=0.000000 0.000000 0.217000 rpy=0.000000 0.5000 3.1415926535897 -> xyz=0.000000 0.000000 0.217000 rpy=0.000000 0.8000 3.1415926535897
- joint j5: origin xyz=0.000000 0.000000 0.217003 rpy=0.000000 0.00 0.000000 -> xyz=0.000000 0.000000 0.217003 rpy=0.000000 0.50 0.000000

Commit message: edited urdf

File: project/kuka_iiwa.urdf (robot description, URDF)
Before this commit: robot kuka_iiwa, 8 links, 7 joints
Links:
- link link6: geometry collision mesh filename=../../../model/iiwa7/meshes/launcher1.obj scale=10 10 10; collision mesh filename=../../../model/iiwa7/meshes/link6.obj scale=1 1 1

Commit message: edited collision

File: project/kuka_iiwa.urdf (robot description, URDF)
Before this commit: robot kuka_iiwa, 8 links, 7 joints
Links:
- link link6: geometry collision mesh filename=../../../model/iiwa7/meshes/launcher_box.obj scale=10 10 10; collision mesh filename=../../../model/iiwa7/meshes/link6.obj scale=1 1 1

Commit message: edited controller and urdfs for robot basketball

File: project/kuka_iiwa.urdf (robot description, URDF)
Before this commit: robot kuka_iiwa, 8 links, 7 joints
Links:
- added link link7, mass 0.00001; visual box size=1 1 0.15
- link link6: geometry collision mesh filename=../../../model/iiwa7/meshes/torus.obj scale=7 7 7; visual mesh filename=../../../model/iiwa7/meshes/hand.obj scale=0.32 0.32 0.32

File: project/mmp_panda.urdf (robot description, URDF)
Before this commit: robot mmp_panda, 11 links, 10 joints
Joints:
- joint joint1: origin xyz=0 0 0.333 rpy=0 0 1.5708 -> xyz=0 0 0.333 rpy=0 0 0.785398

Commit message: edited state machine for shooter and hoop

File: project/kuka_iiwa.urdf (robot description, URDF)
Before this commit: robot kuka_iiwa, 9 links, 7 joints
Links:
- link link7: mass 0.00001 -> 10

Commit message: edit wake up mode

File: project/kuka_iiwa.urdf (robot description, URDF)
Before this commit: robot kuka_iiwa, 9 links, 7 joints
Links:
- link link6: geometry collision mesh filename=../../../model/iiwa7/meshes/torus.obj scale=10 10 10; visual mesh filename=../../../model/iiwa7/meshes/hand.obj scale=0.32 0.32 0.32

Commit message: adjust kuka posture

File: project/kuka_iiwa.urdf (robot description, URDF)
Before this commit: robot kuka_iiwa, 10 links, 9 joints
Joints:
- joint j1: origin xyz=0.000000 0.000000 0.182500 rpy=0.000000 -0.800000 0.000000 -> xyz=0.000000 0.000000 0.182500 rpy=0.000000 -0.700000 0.000000
- joint j3: origin xyz=0.000000 0.000000 0.217000 rpy=0.000000 0.8000 3.1415926535897 -> xyz=0.000000 0.000000 0.217000 rpy=0.000000 0.7000 3.1415926535897
- joint j5: origin xyz=0.000000 0.000000 0.217003 rpy=0.000000 0.50 0.000000 -> xyz=0.000000 0.000000 0.217003 rpy=0.000000 0.30 0.000000

File: project/kuka_iiwa1.urdf (robot description, URDF)
Before this commit: robot kuka_iiwa, 9 links, 7 joints
Joints:
- joint j1: origin xyz=0.000000 0.000000 0.182500 rpy=0.000000 -0.800000 0.000000 -> xyz=0.000000 0.000000 0.182500 rpy=0.000000 -1.500000 0.000000
- joint j3: origin xyz=0.000000 0.000000 0.217000 rpy=0.000000 0.8000 3.1415926535897 -> xyz=0.000000 0.000000 0.217000 rpy=0.000000 1.5000 3.1415926535897
- joint j5: origin xyz=0.000000 0.000000 0.217003 rpy=0.000000 0.50 0.000000 -> xyz=0.000000 0.000000 0.217003 rpy=0.000000 1.20 0.000000

Commit message: edited collision to fit hand

File: project/kuka_iiwa.urdf (robot description, URDF)
Before this commit: robot kuka_iiwa, 10 links, 9 joints
Links:
- link link6: geometry collision box size=.3 .3 0.05; visual mesh filename=../../../model/iiwa7/meshes/hand.obj scale=0.32 0.32 0.32
- link link7: geometry collision box size=.3 .3 0.04; collision box size=0.3 0.3 0.02
- link link8: geometry collision box size=0.3 0.3 0.02
