Commit message: changes to urdfs

File: project/mmp_panda.urdf (robot description, URDF)
Before this commit: robot mmp_panda, 11 links, 10 joints
Links:
- link base_link: geometry visual mesh filename=../../../model/mmp_panda/meshes/visual/panda_BaseCombo.obj

Commit message: added collision to the board and added reset functio to controller

File: project/mmp_panda.urdf (robot description, URDF)
Before this commit: robot mmp_panda, 11 links, 10 joints
Links:
- link link7: geometry collision mesh filename=../../../model/panda/meshes/visual/board.obj scale=0.6 0.6 0.6; visual mesh filename=../../../model/panda/meshes/visual/board.obj scale=0.6 0.6 0.6

Commit message: change to the ideal panda working posture

File: project/mmp_panda.urdf (robot description, URDF)
Before this commit: robot mmp_panda, 11 links, 10 joints
Joints:
- joint joint1: origin xyz=0 0 0.333 rpy=0 0 4.71239 -> xyz=0 0 0.333 rpy=0 0 1.5708
- joint joint6: origin xyz=0 0 0 rpy=1.57079632679 -1.57079632679 0 -> xyz=0 0 0 rpy=1.57079632679 0 0

Commit message: test coordinate

File: project/mmp_panda.urdf (robot description, URDF)
Before this commit: robot mmp_panda, 11 links, 10 joints
Links:
- link base_link: geometry visual mesh filename=../../../model/mmp_panda/meshes/visual/panda_BaseCombo.obj
- link link7: geometry visual mesh filename=../../../model/panda/meshes/visual/board.obj scale=0.6 0.6 0.6; visual mesh filename=../../../model/panda/meshes/visual/link7.obj

Commit message: can follow the predicted position

File: project/mmp_panda.urdf (robot description, URDF)
Before this commit: robot mmp_panda, 11 links, 10 joints
Links:
- link base_link: geometry collision box size=0.4 0.4 0.2; visual mesh filename=../../../model/mmp_panda/meshes/visual/panda_BaseCombo.obj
- link link7: geometry collision mesh filename=../../../model/panda/meshes/visual/board.obj scale=0.6 0.6 0.6; visual mesh filename=../../../model/panda/meshes/visual/board.obj scale=0.6 0.6 0.6

Commit message: it worksgit statusgit status

File: project/mmp_panda.urdf (robot description, URDF)
Before this commit: robot mmp_panda, 11 links, 10 joints
Links:
- link base_link: mass 64.6 -> 10
- link base_x: mass 0.001 -> 0.0001
- link base_y: mass 0.001 -> 0.0001
- link ground_link: mass 0.001 -> 0.0001
- link link1: mass 4 -> 0.01
- link link2: mass 3 -> 0.01
- link link3: mass 3 -> 0.01
- link link4: mass 3 -> 0.01
- link link5: mass 3 -> 0.01
- link link6: mass 2 -> 0.01
- link link7: mass 3.0 -> 0.01; geometry collision mesh filename=../../../model/panda/meshes/visual/board.obj scale=0.6 0.6 0.6; visual mesh filename=../../../model/panda/meshes/visual/board.obj scale=0.6 0.6 0.6

Commit message: let's go target

File: project/mmp_panda.urdf (robot description, URDF)
Before this commit: robot mmp_panda, 11 links, 10 joints
Links:
- link base_link: geometry collision box size=0.4 0.4 0.2; visual mesh filename=../../../model/mmp_panda/meshes/visual/panda_BaseCombo.obj
